Commit message: add MIP with incline with LQR controller

File: rsc/camel_momentum_inverted_pendulum_with_incline.urdf (robot description, URDF)
Before this commit: robot camel_momentum_inverted_pendulum, 4 links, 3 joints
Links:
- added link base-incline; visual cylinder length=0.02 radius=0.005
- added link incline, mass 1.0; collision box size=0.1 0.1 0.0015; visual box size=0.1 0.1 0.0015
Joints:
- added joint fixed-base: type fixed, parent incline, child base
- added joint incline-roll: type revolute, parent base-incline, child incline, origin xyz=0 0.0 0.00075 rpy=0 0 0, axis 1 0 0
- joint base-roll: origin xyz=0 0 0.01275 rpy=0 0 0 -> xyz=0 0.08 0.01275 rpy=0 0 0
- joint fixed_world: child base -> base-incline
