Commit message: joyStick accel generate

File: rsc/camel_wheeledRobot.urdf (robot description, URDF)
Before this commit: robot smb, 8 links, 7 joints
Links:
- removed link lidar
Joints:
- removed joint lidar
- joint LF_WHEEL: limit effort=65 velocity=25 -> effort=65 velocity=90
- joint LH_WHEEL: limit effort=65 velocity=25 -> effort=65 velocity=90
- joint RF_WHEEL: limit effort=65 velocity=25 -> effort=65 velocity=90
- joint RH_WHEEL: limit effort=65 velocity=25 -> effort=65 velocity=90
