Commit message: finish one

File: rsc/camel_hard_IceCream.urdf (robot description, URDF)
Before this commit: robot camel_momentum_inverted_pendulum, 4 links, 3 joints
Links:
- link body: geometry visual box size=0.3 0.1 0.1
Joints:
- joint base-pitch: type continuous -> revolute
- joint hip-pitch: limit (none) -> velocity=17; origin xyz=0.0 0.01 0.35 rpy=0 0 0 -> xyz=0.0 0.0 0.35 rpy=0 0 0

Commit message: edited urdfs more reasonably

File: rsc/camel_hard_IceCream.urdf (robot description, URDF)
Before this commit: robot camel_hard_IceCream, 5 links, 4 joints
Joints:
- joint fixed_body: origin xyz=0.14 0.0 0.04 rpy=0.0 0.0 0.0 -> xyz=0.15 0.0 0.0 rpy=0.0 0.0 0.0

Commit message: edited hard_IceCream urdf to fix bug

File: rsc/camel_hard_IceCream.urdf (robot description, URDF)
Before this commit: robot camel_hard_IceCream, 5 links, 4 joints
Links:
- removed link body_rod
Joints:
- removed joint fixed_body
- joint hip-pitch: child body_rod -> body

Commit message: edit urdf for more likely canine

File: rsc/camel_hard_IceCream.urdf (robot description, URDF)
Before this commit: robot camel_hard_IceCream, 4 links, 3 joints
Links:
- link body: mass 2.5 -> 3.5215; geometry collision box size=0.482 0.122265 0.111; visual box size=0.482 0.122265 0.111
- link rod: mass 1.2 -> 2.179; geometry collision box size=0.003 0.002 0.398372; visual box size=0.03 0.02 0.398372
Joints:
- joint hip-pitch: origin xyz=0.0 0.0 0.35 rpy=0.0 0.0 0.0 -> xyz=0.0 0.0 0.398372 rpy=0.0 0.0 0.0

Commit message: delete velocity limit in hip-pitch for urdfReader

File: rsc/camel_hard_IceCream.urdf (robot description, URDF)
Before this commit: robot camel_hard_IceCream, 4 links, 3 joints
Joints:
- joint hip-pitch: limit velocity=17 -> (none)
