Commit message: solve the bug somehow

File: rsc/camel_double_bar_IceCream.urdf (robot description, URDF)
Before this commit: robot camel_momentum_inverted_pendulum, 5 links, 4 joints
Links:
- link calf: geometry collision box size=0.003 0.002 0.2; visual box size=0.03 0.02 0.2

File: rsc/camel_hard_IceCream.urdf (robot description, URDF)
Before this commit: robot camel_momentum_inverted_pendulum, 4 links, 3 joints
Links:
- added link body_rod; visual sphere radius=0.01
- link base: mass None -> 0.01
- link rod: geometry collision box size=0.003 0.002 0.35; visual box size=0.03 0.02 0.35
Joints:
- added joint fixed_body: type fixed, parent body_rod, child body, origin xyz=0.14 0.0 0.04 rpy=0.0 0.0 0.0
- joint hip-pitch: child body -> body_rod; origin xyz=0.0 0.0 0.35 rpy=0 0 0 -> xyz=0.0 0.0 0.35 rpy=0.0 0.0 0.0

Commit message: edit parameter to fit canine

File: rsc/camel_double_bar_IceCream.urdf (robot description, URDF)
Before this commit: robot camel_momentum_inverted_pendulum, 5 links, 4 joints
Links:
- link body: mass 2.5 -> 5.0075; geometry collision box size=0.482 0.122265 0.111; visual box size=0.482 0.122265 0.111
- link calf: mass 0.2 -> 0.207; geometry collision box size=0.003 0.002 0.2; visual box size=0.03 0.02 0.23
- link thigh: mass 0.2 -> 1.229; geometry visual box size=0.03 0.02 0.23
Joints:
- joint hip-pitch: origin xyz=0.0 0.0 0.2 rpy=0 0 0 -> xyz=0.0 0.0 0.23 rpy=0 0 0
- joint knee-pitch: origin xyz=0 0 0.2 rpy=0 0 0 -> xyz=0 0 0.23 rpy=0 0 0
