Commit message: reset cha branch

File: rsc/obstacle.urdf (robot description, URDF)
Before this commit: robot obstacle, 4 links, 3 joints
Joints:
- joint base: origin xyz=5 0 0 rpy=0 0 0 -> xyz=2 -0.05 0 rpy=0 0 0

Commit message: Apply external torque observer to Canine.

File: rsc/obstacle.urdf (robot description, URDF)
Before this commit: robot obstacle, 4 links, 3 joints
Joints:
- joint base: origin xyz=2 -0.05 0 rpy=0 0 0 -> xyz=-0.5 -0.05 0 rpy=0 0 0
