Commit message: initialize DongDog branch

File: rsc/camel_dong_dog/camel_dong_dog_one_leg.urdf (robot description, URDF)
Before this commit: robot camel_dong_dog, 7 links, 7 joints
Links:
- link base: mass None -> 10; geometry visual box size=0.25 0.25 2.5
- link calf1: mass None -> 3.0
- link calf2: mass None -> 3.0
- link calf3: mass None -> 3.0
- link shoulder: mass None -> 3.0
- link thigh: mass None -> 3.0
Joints:
- joint J1: axis 0 -1 0 -> 1 0 0; origin xyz=0 0 1 rpy=0 0 0 -> xyz=0 0 0 rpy=0 0 0
- joint J2: axis (none) -> 1 0 0
- joint J3: axis (none) -> 1 0 0; parent calf2 -> shoulder
- joint J4: child calf3 -> calf2; parent shoulder -> calf3
- joint J5: child calf2 -> calf1; parent calf3 -> calf2
- joint base: axis 0 0 0 -> 0 0 1; origin xyz=0 0 0 rpy=0 0 0 -> xyz=0 -0.025 0.0 rpy=0 0 0

Commit message: initialize DongDog branch

File: rsc/camel_dong_dog/camel_dong_dog_one_leg.urdf (robot description, URDF)
Before this commit: robot camel_dong_dog, 7 links, 7 joints
Links:
- link base: geometry visual box size=0.25 0.25 1

Commit message: initialize DongDog branch

File: rsc/camel_dong_dog/camel_dong_dog_one_leg.urdf (robot description, URDF)
Before this commit: robot camel_dong_dog, 7 links, 7 joints
Links:
- removed link calf1
- removed link calf2
- removed link calf3
- added link calf, mass 3.0; visual mesh filename=calf.stl
Joints:
- removed joint J3
- removed joint J4
- removed joint J5
- joint J2: child calf1 -> calf

Commit message: initialize DongDog branch

File: rsc/camel_dong_dog/camel_dong_dog_one_leg.urdf (robot description, URDF)
Before this commit: robot camel_dong_dog, 5 links, 4 joints
Links:
- link base: geometry visual box size=0.25 0.25 2.5
Joints:
- joint J1: origin xyz=0 0 0 rpy=0 0 0 -> xyz=-0.25 0.475 0.2 rpy=0 0 0
- joint J2: origin xyz=0 0 0 rpy=0 0 0 -> xyz=-0.075 -0.725 -0.725 rpy=0 0 0
- joint base: origin xyz=0 -0.025 0.0 rpy=0 0 0 -> xyz=-0.25 0 -0.3 rpy=0 0 0
