Commit message: initialize DongDog branch

File: rsc/camel_dong_dog_full/camel_dong_dog_full.urdf (robot description, URDF)
Before this commit: robot camel_dong_dog, 2 links, 1 joints
Links:
- added link body, mass 3.0; visual mesh filename=Body.stl
- link base: mass 10 -> 3.0; geometry visual box size=0.025 0.025 2.5
Joints:
- added joint base: type prismatic, parent base, child body, origin xyz=0 0 0 rpy=0 0 0, axis 0 0 1

Commit message: initialize DongDog branch

File: rsc/camel_dong_dog_full/camel_dong_dog_full.urdf (robot description, URDF)
Before this commit: robot camel_dong_dog, 3 links, 2 joints
Links:
- link base: mass 3.0 -> 1
- link body: mass 3.0 -> 1; geometry visual mesh filename=Body.stl.stl scale=0.5 0.5 0.5
Joints:
- joint base: origin xyz=0 0 0 rpy=0 0 0 -> xyz=-0.25 0 -0.3 rpy=0 0 0

Commit message: initialize DongDog branch

File: rsc/camel_dong_dog_full/camel_dong_dog_full.urdf (robot description, URDF)
Before this commit: robot camel_dong_dog, 3 links, 2 joints
Links:
- removed link body
- added link calf, mass 3.0; visual mesh filename=calf.stl
- added link shoulder, mass 3.0; visual mesh filename=shoulder.stl
- added link thigh, mass 3.0; visual mesh filename=thigh.stl
- link base: mass 1 -> 10; geometry visual box size=0.25 0.25 2.5
Joints:
- added joint J1: type revolute, parent shoulder, child thigh, origin xyz=-0.25 0.475 0.2 rpy=0 0 0, axis 1 0 0
- added joint J2: type revolute, parent thigh, child calf, origin xyz=-0.075 -0.725 -0.725 rpy=0 0 0, axis 1 0 0
- joint base: child body -> shoulder

Commit message: initialize dondDog branch

File: rsc/camel_dong_dog_full/camel_dong_dog_full.urdf (robot description, URDF)
Before this commit: robot camel_dong_dog, 3 links, 2 joints
Links:
- link body: mass 3.0 -> 1.0
