Commit message: temporary urdf

File: rsc/camel_two_leg/camel_two_leg.urdf (robot description, URDF)
Before this commit: robot camel_two_leg_bot, 2 links, 1 joints
Links:
- removed link world
- added link hip_1, mass 0.7835; collision cylinder length=0.034 radius=0.049; visual mesh filename=base_link.STL
- added link trunk, mass 4.713; collision box size=0.267 0.194 0.114; visual box size=0.267 0.194 0.114
Joints:
- removed joint base_static_joint
- added joint R-hip-joint: type revolute, parent base, child hip_1, origin xyz=0 -0.08505 0 rpy=0 0 0, axis 0 1 0
- added joint floating_base: type fixed, parent base, child trunk, origin xyz=0 0 0 rpy=0 0 0

Commit message: adding urdf for two legged robot with floating base

File: rsc/camel_two_leg/camel_two_leg.urdf (robot description, URDF)
Before this commit: robot camel_two_leg_bot, 3 links, 2 joints
Links:
- removed link base
- removed link hip_1
- added link BL-hip, mass 0.8; collision cylinder length=0.03 radius=0.05; visual cylinder length=0.03 radius=0.05
- added link BL_foot, mass 0.06; collision sphere radius=0.02; visual sphere radius=0.01
- added link BL_lower_leg, mass 0.2; collision box size=0.03 0.02 0.2; visual box size=0.03 0.02 0.2
- added link BL_upper_leg, mass 0.2; collision box size=0.03 0.02 0.2; visual box size=0.03 0.02 0.2
- added link BR-hip, mass 0.8; collision cylinder length=0.03 radius=0.05; visual cylinder length=0.03 radius=0.05
- added link BR_foot, mass 0.06; collision sphere radius=0.02; visual sphere radius=0.01
- added link BR_lower_leg, mass 0.2; collision box size=0.03 0.02 0.2; visual box size=0.03 0.02 0.2
- added link BR_upper_leg, mass 0.2; collision box size=0.03 0.02 0.2; visual box size=0.03 0.02 0.2
- link trunk: mass 4.713 -> 5.0; geometry collision box size=0.3 0.2 0.1; visual box size=0.3 0.2 0.1
Joints:
- removed joint R-hip-joint
- removed joint floating_base
- added joint BL-hip-pitch: type revolute, parent trunk, child BL-hip, origin xyz=-0.1 0.115 0 rpy=0 0 0, axis 0 1 0
- added joint BL-knee-pitch: type revolute, parent BL_upper_leg, child BL_lower_leg, origin xyz=0 0 -0.1 rpy=0 0 0, axis 0 1 0
- added joint BL-upper-leg: type fixed, parent BL-hip, child BL_upper_leg, origin xyz=0 0 -0.1 rpy=0 0 0
- added joint BL_foot_fixed: type fixed, parent BL_lower_leg, child BL_foot, origin xyz=0 0 -0.2 rpy=0 0 0
- added joint BR-hip-pitch: type revolute, parent trunk, child BR-hip, origin xyz=-0.1 -0.115 0 rpy=0 0 0, axis 0 1 0
- added joint BR-knee-pitch: type revolute, parent BR_upper_leg, child BR_lower_leg, origin xyz=0 0 -0.1 rpy=0 0 0, axis 0 1 0
- added joint BR-upper-leg: type fixed, parent BR-hip, child BR_upper_leg, origin xyz=0 0 -0.1 rpy=0 0 0
- added joint BR_foot_fixed: type fixed, parent BR_lower_leg, child BR_foot, origin xyz=0 0 -0.2 rpy=0 0 0
