Commit message: modify collision body

File: rsc/camel_JHdog_single_leg/JHdog_single_leg.urdf (robot description, URDF)
Before this commit: robot JHdog-single-leg, 7 links, 6 joints
Links:
- removed link foot
- removed link hip_2
- link hip_1: geometry collision cylinder length=0.12 radius=0.038; visual mesh filename=hip.STL
- link lower_leg: geometry collision box size=0.03 0.025 0.207; visual mesh filename=calf.STL
- link upper_leg: geometry collision box size=0.035 0.04 0.22; visual mesh filename=thigh.STL
Joints:
- removed joint ankle_pitch
- removed joint hip_upper
- joint hip_pitch: child hip_2 -> upper_leg; origin xyz=0 -0.080 0.0 rpy=0 0 0 -> xyz=0 -0.03 0.0 rpy=0 0 0
- joint knee_pitch: origin xyz=0 0 -0.15 rpy=0 0 0 -> xyz=0 -0.064 -0.18 rpy=0 0 0
